Commit message: update robot for gazebo_classic

File: robotaksi_classic/urdf/robotaksi.urdf.xacro (robot description, xacro)
@@ -14,5 +14,5 @@
         <visual>
             <geometry>
-                <mesh filename="package://robotaksi_description/meshes/robotaksi.dae" />
+                <mesh filename="package://robotaksi_classic/meshes/robotaksi.dae" />
             </geometry>
             <origin xyz="0 0 ${base_height / 2.0}" rpy="0 0 0" />
