Commit message: change file paths

File: urdf_classic/robotaksi.urdf.xacro (robot description, xacro)
@@ -14,5 +14,5 @@
         <visual>
             <geometry>
-                <mesh filename="package://robotaksi_classic/meshes/robotaksi.dae" />
+                <mesh filename="package://robotaksi_autonomous_car/meshes/robotaksi.dae" />
             </geometry>
             <origin xyz="0 0 ${base_height / 2.0}" rpy="0 0 0" />

File: urdf_harmonic/robotaksi.urdf.xacro (robot description, xacro)
@@ -14,5 +14,5 @@
         <visual>
             <geometry>
-                <mesh filename="package://simulation_2025/meshes/robotaksi.dae" />
+                <mesh filename="package://robotaksi_autonomous_car/meshes/robotaksi.dae" />
             </geometry>
             <origin xyz="0 0 ${base_height / 2.0}" rpy="0 0 0" />
